Commit message: Start.

File: src/robot_tutorial/urdf/macro.xacro (robot description, xacro)
@@ -35,5 +35,5 @@
     <inertia ixx="${mass*(3*r*r+l*l)/12}" ixy = "0" ixz = "0" iyy="${mass*(3*r*r+l*l)/12}" iyz = "0" izz="${mass*(r*r)/2}" />
   </xacro:macro>
-  <macro name="box_inertia" params="m x y z">
+  <!-- <macro name="box_inertia" params="m x y z">
     <inertia  ixx="${m*(y*y+z*z)/12}" ixy = "0" ixz = "0"
       iyy="${m*(x*x+z*z)/12}" iyz = "0"
@@ -46,4 +46,4 @@
       izz="${2*m*r*r/5}"
     />
-  </macro>
+  </macro> -->
 </robot>

File: src/robot_tutorial/urdf/robot.xacro (robot description, xacro)
@@ -12,5 +12,5 @@
     <inertial>
       <mass value="27.875"/>
-      <origin rpy="0 0 0" xyz="0 0 0.1"/>
+      <origin rpy="5 -8 0" xyz="0 0 0.1"/>
       <inertia ixx="1.121e+0" ixy="3.55909983e-9" ixz="-9.359e-8" iyy="1.121e+0" iyz="-3.899e-9" izz="1.816e-1"/>
     </inertial>
@@ -22,4 +22,5 @@
     <visual>
       <origin xyz="5 -8 0" rpy="0 0 0" />
+      <!-- <origin xyz="0 0 0" rpy="0 0 0" /> -->
       <geometry>
 	      <mesh filename="package://robot_tutorial/mesches/body_yes.dae" />
@@ -27,4 +28,16 @@
     </visual>
   </link>
+  <!-- Create wheel right -->
+  <!-- <xacro:link_wheel name="link_rightA_wheel"/>
+  <xacro:joint_wheel name="joint_rightA_wheel" parent="robot_body"  child="link_rightA_wheel"  origin_xyz="-0.1 -0.235 -0.326"  /> -->
+  <!-- Create wheel right -->
+  <!-- <xacro:link_wheel name="link_rightB_wheel"/>
+  <xacro:joint_wheel name="joint_rightB_wheel" parent="robot_body"   child="link_rightB_wheel"   origin_xyz="0.1 -0.235 -0.326"  /> -->
+  <!-- Left Wheel link -->
+  <!-- <xacro:link_wheel name="link_leftA_wheel"/>
+  <xacro:joint_wheel name="joint_leftA_wheel" parent="robot_body"   child="link_leftA_wheel"   origin_xyz="-0.1 0.215 -0.326"  /> -->
+  <!-- Left Wheel link -->
+  <!-- <xacro:link_wheel name="link_leftB_wheel"/>
+  <xacro:joint_wheel name="joint_leftB_wheel" parent="robot_body"   child="link_leftB_wheel"   origin_xyz="0.1 0.215 -0.326"  /> -->
   <!-- Create wheel right -->
   <xacro:link_wheel name="link_rightA_wheel"/>

Commit message: Test move robot.

File: src/robot_tutorial/urdf/macro.xacro (robot description, xacro)
@@ -35,5 +35,5 @@
     <inertia ixx="${mass*(3*r*r+l*l)/12}" ixy = "0" ixz = "0" iyy="${mass*(3*r*r+l*l)/12}" iyz = "0" izz="${mass*(r*r)/2}" />
   </xacro:macro>
-  <!-- <macro name="box_inertia" params="m x y z">
+  <macro name="box_inertia" params="m x y z">
     <inertia  ixx="${m*(y*y+z*z)/12}" ixy = "0" ixz = "0"
       iyy="${m*(x*x+z*z)/12}" iyz = "0"
@@ -46,4 +46,4 @@
       izz="${2*m*r*r/5}"
     />
-  </macro> -->
+  </macro>
 </robot>

File: src/robot_tutorial/urdf/robot.xacro (robot description, xacro)
@@ -29,19 +29,7 @@
   </link>
   <!-- Create wheel right -->
-  <!-- <xacro:link_wheel name="link_rightA_wheel"/>
-  <xacro:joint_wheel name="joint_rightA_wheel" parent="robot_body"  child="link_rightA_wheel"  origin_xyz="-0.1 -0.235 -0.326"  /> -->
-  <!-- Create wheel right -->
-  <!-- <xacro:link_wheel name="link_rightB_wheel"/>
-  <xacro:joint_wheel name="joint_rightB_wheel" parent="robot_body"   child="link_rightB_wheel"   origin_xyz="0.1 -0.235 -0.326"  /> -->
-  <!-- Left Wheel link -->
-  <!-- <xacro:link_wheel name="link_leftA_wheel"/>
-  <xacro:joint_wheel name="joint_leftA_wheel" parent="robot_body"   child="link_leftA_wheel"   origin_xyz="-0.1 0.215 -0.326"  /> -->
-  <!-- Left Wheel link -->
-  <!-- <xacro:link_wheel name="link_leftB_wheel"/>
-  <xacro:joint_wheel name="joint_leftB_wheel" parent="robot_body"   child="link_leftB_wheel"   origin_xyz="0.1 0.215 -0.326"  /> -->
-  <!-- Create wheel right -->
   <xacro:link_wheel name="link_rightA_wheel"/>
   <xacro:joint_wheel name="joint_rightA_wheel" parent="robot_body"  child="link_rightA_wheel"  origin_xyz="4.9 -8.235 -0.326"  />
-  <!-- Left Wheel link -->
+  <!-- Create wheel right -->
   <xacro:link_wheel name="link_rightB_wheel"/>
   <xacro:joint_wheel name="joint_rightB_wheel" parent="robot_body"   child="link_rightB_wheel"   origin_xyz="5.1 -8.235 -0.326"  />
@@ -52,5 +40,5 @@
   <xacro:link_wheel name="link_leftB_wheel"/>
   <xacro:joint_wheel name="joint_leftB_wheel" parent="robot_body"   child="link_leftB_wheel"   origin_xyz="5.1 -7.785 -0.326"  />
-  <!-- <link name="sensor_laser">
+  <link name="sensor_laser">
     <xacro:cylinder_inertia mass="1" r="0.05" l="0.1" />
     <visual>
@@ -72,7 +60,7 @@
     <parent link="robot_body"/>
     <child link="sensor_laser"/>
-  </joint> -->
+  </joint>
   <!-- Camera -->
-  <!-- <link name="camera">
+  <link name="camera">
     <collision>
       <origin xyz="0 0 0" rpy="0 0 0"/>
@@ -82,5 +70,5 @@
     </collision>
     <visual>
-      <origin xyz="5.1 -8 0.41" rpy="0 0 0"/>
+      <origin xyz="0 0 0" rpy="0 0 0"/>
       <geometry>
         <box size="${cameraSize} ${cameraSize} ${cameraSize}"/>
@@ -96,7 +84,7 @@
   <joint name="joint_robot_to_camera" type="fixed">
     <axis xyz="0.0 1.0 0.0"/>
-    <origin xyz="0 0 0 " rpy="0.0 0.0 0.0"/>
+    <origin  xyz="5.1 -8 0.41" rpy="0.0 0.0 0.0"/>
     <parent link="robot_body"/>
     <child link="camera"/>
-  </joint> -->
+  </joint>
 </robot>
