Commit message: Robot complet.

File: src/robot_tutorial/urdf/robot.xacro (robot description, xacro)
@@ -12,5 +12,5 @@
     <inertial>
       <mass value="27.875"/>
-      <origin rpy="5 -8 0" xyz="0 0 0.1"/>
+      <origin rpy="0 0 0" xyz="5 -8 0"/>
       <inertia ixx="1.121e+0" ixy="3.55909983e-9" ixz="-9.359e-8" iyy="1.121e+0" iyz="-3.899e-9" izz="1.816e-1"/>
     </inertial>

Commit message: Update repository.

File: src/robot_tutorial/urdf/robot.xacro (robot description, xacro)
@@ -3,14 +3,18 @@
   <xacro:property name = "cameraSize" value = "0.05" />
   <xacro:property name = "cameraMass" value = "0.1" />
+  <xacro:arg name="gpu" default="false"/>
+  <xacro:property name="gpu" value="$(arg gpu)" />
   <!-- include the xacro files-->
   <xacro:include filename="$(find robot_tutorial)/urdf/materials.xacro"/>
   <xacro:include filename="$(find robot_tutorial)/urdf/robot.gazebo"/>
   <xacro:include filename="$(find robot_tutorial)/urdf/macro.xacro" />
+  <link name="base_link">
+  </link>
   <link name="robot_body">
     <!-- pose and inertial -->
     <pose>0 0 0.1 0 0 0</pose>
     <inertial>
+     <origin xyz="0 0 0" rpy="0 0 0" />
       <mass value="27.875"/>
-      <origin rpy="5 -8 0" xyz="0 0 0.1"/>
       <inertia ixx="1.121e+0" ixy="3.55909983e-9" ixz="-9.359e-8" iyy="1.121e+0" iyz="-3.899e-9" izz="1.816e-1"/>
     </inertial>
@@ -21,6 +25,5 @@
     </collision>
     <visual>
-      <origin xyz="5 -8 0" rpy="0 0 0" />
-      <!-- <origin xyz="0 0 0" rpy="0 0 0" /> -->
+      <origin xyz="0 0 0" rpy="0 0 0" />
       <geometry>
 	      <mesh filename="package://robot_tutorial/mesches/body_yes.dae" />
@@ -28,37 +31,26 @@
     </visual>
   </link>
+  <joint name="joint_base_link_to_robot" type="fixed">
+    <origin xyz="0.0 0.0 0.0" rpy="0.0 0.0 0.0"/>
+    <parent link="base_link"/>
+    <child link="robot_body"/>
+  </joint>
   <!-- Create wheel right -->
   <xacro:link_wheel name="link_rightA_wheel"/>
-  <xacro:joint_wheel name="joint_rightA_wheel" parent="robot_body"  child="link_rightA_wheel"  origin_xyz="4.9 -8.235 -0.326"  />
+  <xacro:joint_wheel name="joint_rightA_wheel" parent="robot_body"  child="link_rightA_wheel"  origin_xyz="-0.1 0.215 -0.326"  />
   <!-- Create wheel right -->
   <xacro:link_wheel name="link_rightB_wheel"/>
-  <xacro:joint_wheel name="joint_rightB_wheel" parent="robot_body"   child="link_rightB_wheel"   origin_xyz="5.1 -8.235 -0.326"  />
+  <xacro:joint_wheel name="joint_rightB_wheel" parent="robot_body"   child="link_rightB_wheel"   origin_xyz="0.1 0.215 -0.326"  />
   <!-- Left Wheel link -->
   <xacro:link_wheel name="link_leftA_wheel"/>
-  <xacro:joint_wheel name="joint_leftA_wheel" parent="robot_body"   child="link_leftA_wheel"   origin_xyz="4.9 -7.785 -0.326"  />
+  <xacro:joint_wheel name="joint_leftA_wheel" parent="robot_body"   child="link_leftA_wheel"   origin_xyz="-0.1 -0.238 -0.326"  />
   <!-- Left Wheel link -->
   <xacro:link_wheel name="link_leftB_wheel"/>
-  <xacro:joint_wheel name="joint_leftB_wheel" parent="robot_body"   child="link_leftB_wheel"   origin_xyz="5.1 -7.785 -0.326"  />
-  <link name="sensor_laser">
-    <xacro:cylinder_inertia mass="1" r="0.05" l="0.1" />
-    <visual>
-      <origin xyz="4.85 -8 0.441" rpy="0 0 0" />
-      <geometry>
-        <cylinder radius="0.05" length="0.1"/>
-      </geometry>
-      <material name="white" />
-    </visual>
-    <collision>
-      <origin xyz="0 0 0" rpy="0 0 0"/>
-      <geometry>
-        <cylinder radius="0.05" length="0.1"/>
-      </geometry>
-    </collision>
-  </link>
-  <joint name="joint_robot_to_sensor_laser" type="fixed">
-    <origin xyz="0.15 0 0.05" rpy="0 0 0"/>
-    <parent link="robot_body"/>
-    <child link="sensor_laser"/>
-  </joint>
+  <xacro:joint_wheel name="joint_leftB_wheel" parent="robot_body"   child="link_leftB_wheel"   origin_xyz="0.1 -0.238 -0.326"  />
+  <!-- VLP-16 -->
+  <xacro:include filename="$(find velodyne_description)/urdf/VLP-16.urdf.xacro"/>
+  <VLP-16 parent="robot_body" name="velodyne" topic="/velodyne_points" hz="10" samples="440" gpu="${gpu}">
+    <origin xyz="0 0 0.435" rpy="0 0 0" />
+  </VLP-16>
   <!-- Camera -->
   <link name="camera">
@@ -83,6 +75,5 @@
   </link>
   <joint name="joint_robot_to_camera" type="fixed">
-    <axis xyz="0.0 1.0 0.0"/>
-    <origin  xyz="5.1 -8 0.41" rpy="0.0 0.0 0.0"/>
+    <origin  xyz="0.11 0 0.38" rpy="0.0 0.0 0.0"/>
     <parent link="robot_body"/>
     <child link="camera"/>
